Commit message: update tmr_description

File: tmr_description/xacro/macro.materials.xacro (robot description, xacro)
@@ -1,35 +1,38 @@
 <?xml version="1.0"?>
 <robot xmlns:xacro="http://www.ros.org/wiki/xacro">
-	<xacro:macro name="tmr_materials">
+  <xacro:macro name="tmr_materials">
+    <material name="none">
+      <color rgba="0.0 0.0 0.0 1.0" />
+    </material>
     <material name="grey">
-			<color rgba="0.5 0.5 0.5 1.0" />
-		</material>
-		<material name="white">
-			<color rgba="0.95 0.95 0.95 1.0" />
-		</material>
-		<material name="red">
-			<color rgba="0.95 0.0 0.0 1.0" />
-		</material>
-		<material name="orange">
-			<color rgba="1.0 0.5 0.0 1.0" />
-		</material>
-		<material name="yellow">
-			<color rgba="1.0 1.0 0.0 1.0" />
-		</material>
-		<material name="green">
-			<color rgba="0.0 1.0 0.0 1.0" />
-		</material>
-		<material name="blue">
-			<color rgba="0.0 0.0 1.0 1.0" />
-		</material>
-		<material name="indigo">
-			<color rgba="0.3 0.3 0.6 1.0" />
-		</material>
-		<material name="violet">
-			<color rgba="0.6 0.0 1.0 1.0" />
-		</material>
-		<material name="black">
-			<color rgba="0.0 0.0 0.0 1.0" />
-		</material>
-	</xacro:macro>
+      <color rgba="0.5 0.5 0.5 1.0" />
+    </material>
+    <material name="white">
+      <color rgba="0.95 0.95 0.95 1.0" />
+    </material>
+    <material name="red">
+      <color rgba="0.95 0.0 0.0 1.0" />
+    </material>
+    <material name="orange">
+      <color rgba="1.0 0.5 0.0 1.0" />
+    </material>
+    <material name="yellow">
+      <color rgba="1.0 1.0 0.0 1.0" />
+    </material>
+    <material name="green">
+      <color rgba="0.0 1.0 0.0 1.0" />
+    </material>
+    <material name="blue">
+      <color rgba="0.0 0.0 1.0 1.0" />
+    </material>
+    <material name="indigo">
+      <color rgba="0.3 0.3 0.6 1.0" />
+    </material>
+    <material name="violet">
+      <color rgba="0.6 0.0 1.0 1.0" />
+    </material>
+    <material name="black">
+      <color rgba="0.0 0.0 0.0 1.0" />
+    </material>
+  </xacro:macro>
 </robot>

File: tmr_description/xacro/macro.tm5-900-mdh.urdf.xacro (robot description, xacro)
@@ -29,6 +29,6 @@
       </geometry>
     </collision>
-    <xacro:cylinder_inertial_z length="0.05" mass="${mass_0}" radius="0.06">
-      <origin rpy="0 0 0" xyz="0 0 0" />
+    <xacro:cylinder_inertial_z radius="0.06" length="0.05" mass="${mass_0}">
+      <origin xyz="0 0 0" rpy="0 0 0" />
     </xacro:cylinder_inertial_z>
   </link>
@@ -36,7 +36,7 @@
     <parent link="${prefix}link_0" />
     <child link="${prefix}link_1" />
-    <origin rpy="0.000000 -0.000000 -0.000018" xyz="0.000000 0.000000 0.145100" />
+    <origin xyz="0.000000 0.000000 0.145100" rpy="0.000000 -0.000000 -0.000018" />
     <axis xyz="0 0 1" />
-    <limit effort="320.0" lower="-4.8346" upper="4.8346" velocity="3.14" />
+    <limit lower="-4.8346" upper="4.8346" velocity="3.14" effort="320.0" />
   </joint>
   <link name="${prefix}link_1">
@@ -52,6 +52,6 @@
       </geometry>
     </collision>
-    <xacro:cylinder_inertial_z length="0.15" mass="${mass_1}" radius="0.06">
-      <origin rpy="0 0 0" xyz="0 0 0" />
+    <xacro:cylinder_inertial_z radius="0.06" length="0.15" mass="${mass_1}">
+      <origin xyz="0 0 0" rpy="0 0 0" />
     </xacro:cylinder_inertial_z>
   </link>
@@ -59,7 +59,7 @@
     <parent link="${prefix}link_1" />
     <child link="${prefix}link_2" />
-    <origin rpy="-1.208300 -1.569562 -0.362515" xyz="0.000010 0.000068 0.000000" />
+    <origin xyz="0.000010 0.000068 0.000000" rpy="-1.208300 -1.569562 -0.362515" />
     <axis xyz="0 0 1" />
-    <limit effort="320" lower="-3.2638" upper="3.2638" velocity="3.14" />
+    <limit lower="-3.2638" upper="3.2638" velocity="3.14" effort="320" />
   </joint>
   <link name="${prefix}link_2">
@@ -75,6 +75,6 @@
       </geometry>
     </collision>
-    <xacro:cylinder_inertial_x length="0.429" mass="${mass_2}" radius="0.06">
-      <origin rpy="0 0 0" xyz="0.2145 0 -0.146" />
+    <xacro:cylinder_inertial_x radius="0.06" length="0.429" mass="${mass_2}">
+      <origin xyz="0.2145 0 -0.146" rpy="0 0 0" />
     </xacro:cylinder_inertial_x>
   </link>
@@ -82,7 +82,7 @@
     <parent link="${prefix}link_2" />
     <child link="${prefix}link_3" />
-    <origin rpy="0.005376 -0.000593 0.006547" xyz="0.429029 -0.000000 0.000068" />
+    <origin xyz="0.429029 -0.000000 0.000068" rpy="0.005376 -0.000593 0.006547" />
     <axis xyz="0 0 1" />
-    <limit effort="320" lower="-2.8274" upper="2.8274" velocity="3.14" />
+    <limit lower="-2.8274" upper="2.8274" velocity="3.14" effort="320" />
   </joint>
   <link name="${prefix}link_3">
@@ -98,6 +98,6 @@
       </geometry>
     </collision>
-    <xacro:cylinder_inertial_x length="0.4115" mass="${mass_3}" radius="0.045">
-      <origin rpy="0 0 0" xyz="0.20575 0 -0.0163" />
+    <xacro:cylinder_inertial_x radius="0.045" length="0.4115" mass="${mass_3}">
+      <origin xyz="0.20575 0 -0.0163" rpy="0 0 0" />
     </xacro:cylinder_inertial_x>
   </link>
@@ -105,7 +105,7 @@
     <parent link="${prefix}link_3" />
     <child link="${prefix}link_4" />
-    <origin rpy="-0.001062 -0.001154 1.571161" xyz="0.411623 0.000141 -0.122132" />
+    <origin xyz="0.411623 0.000141 -0.122132" rpy="-0.001062 -0.001154 1.571161" />
     <axis xyz="0 0 1" />
-    <limit effort="80" lower="-3.2638" upper="3.2638" velocity="3.92" />
+    <limit lower="-3.2638" upper="3.2638" velocity="3.92" effort="80" />
   </joint>
   <link name="${prefix}link_4">
@@ -121,6 +121,6 @@
       </geometry>
     </collision>
-    <xacro:cylinder_inertial_y length="0.12" mass="${mass_4}" radius="0.045">
-      <origin rpy="0 0 0" xyz="0 0 0" />
+    <xacro:cylinder_inertial_y radius="0.045" length="0.12" mass="${mass_4}">
+      <origin xyz="0 0 0" rpy="0 0 0" />
     </xacro:cylinder_inertial_y>
   </link>
@@ -128,7 +128,7 @@
     <parent link="${prefix}link_4" />
     <child link="${prefix}link_5" />
-    <origin rpy="1.571314 -0.001443 0.000362" xyz="-0.000095 -0.106061 -0.000055" />
+    <origin xyz="-0.000095 -0.106061 -0.000055" rpy="1.571314 -0.001443 0.000362" />
     <axis xyz="0 0 1" />
-    <limit effort="80" lower="-3.2638" upper="3.2638" velocity="3.92" />
+    <limit lower="-3.2638" upper="3.2638" velocity="3.92" effort="80" />
   </joint>
   <link name="${prefix}link_5">
@@ -144,6 +144,6 @@
       </geometry>
     </collision>
-    <xacro:cylinder_inertial_y length="0.12" mass="${mass_5}" radius="0.045">
-      <origin rpy="0 0 0" xyz="0 0 0" />
+    <xacro:cylinder_inertial_y radius="0.045" length="0.12" mass="${mass_5}">
+      <origin xyz="0 0 0" rpy="0 0 0" />
     </xacro:cylinder_inertial_y>
   </link>
@@ -151,7 +151,7 @@
     <parent link="${prefix}link_5" />
     <child link="${prefix}link_6" />
-    <origin rpy="1.571355 -0.011670 0.001437" xyz="0.000183 -0.114320 -0.000064" />
+    <origin xyz="0.000183 -0.114320 -0.000064" rpy="1.571355 -0.011670 0.001437" />
     <axis xyz="0 0 1" />
-    <limit effort="80" lower="-4.8346" upper="4.8346" velocity="3.92" />
+    <limit lower="-4.8346" upper="4.8346" velocity="3.92" effort="80" />
   </joint>
   <link name="${prefix}link_6">
@@ -167,6 +167,6 @@
       </geometry>
     </collision>
-    <xacro:cylinder_inertial_z length="0.06" mass="${mass_6}" radius="0.045">
-      <origin rpy="0 0 0" xyz="0 0 0" />
+    <xacro:cylinder_inertial_z radius="0.045" length="0.06" mass="${mass_6}">
+      <origin xyz="0 0 0" rpy="0 0 0" />
     </xacro:cylinder_inertial_z>
   </link>
@@ -175,5 +175,5 @@
     <parent link="${prefix}base" />
     <child link="${prefix}link_0" />
-    <origin rpy="0.0 0.0 0.0" xyz="0.0 0.0 0.0" />
+    <origin xyz="0.0 0.0 0.0" rpy="0.0 0.0 0.0" />
   </joint>
   <link name="${prefix}flange" />
@@ -181,5 +181,5 @@
     <parent link="${prefix}link_6" />
     <child link="${prefix}flange" />
-    <origin rpy="0.012173 0.024881 0.000303" xyz="-0.000179 0.000000 0.000000" />
+    <origin xyz="-0.000179 0.000000 0.000000" rpy="0.012173 0.024881 0.000303" />
   </joint>
 <!--LinkDescription-->
