Commit message: change collision(xarco) to use compound shape instead mesh

File: tmr_description/xacro/macro.tm5-900-capsule.urdf.xacro (robot description, xacro)
@@ -24,9 +24,4 @@
       <material name="${color}" />
     </visual>
-    <!--collision>
-      <geometry>
-        <mesh filename="package://tmr_description/meshes/tm5-900/collision/tm5_base_c.stl" />
-      </geometry>
-    </collision-->
     <collision>
       <geometry>
@@ -54,20 +49,21 @@
       <material name="${color}" />
     </visual>
-    <!--collision>
-      <geometry>
-        <mesh filename="package://tmr_description/meshes/tm5-900/collision/tmr_400w_01_c.stl" />
-      </geometry>
-    </collision-->
-    <collision>
-      <geometry>
-        <cylinder length="0.16" radius="0.064" />
-      </geometry>
-      <origin xyz="0 0 -0.001" rpy="0 0 0" />
-    </collision>
-    <collision>
-      <geometry>
-        <cylinder length="0.066" radius="0.064" />
-      </geometry>
-      <origin xyz="0 -0.033 0" rpy="${-0.5*pi} 0 0" />
+    <collision>
+      <geometry>
+        <cylinder length="0.13" radius="0.064" />
+      </geometry>
+      <origin xyz="0 0 -0.016" rpy="0 0 0" />
+    </collision>
+    <collision>
+      <geometry>
+        <sphere radius="0.064" />
+      </geometry>
+      <origin xyz="0 0 -0.081" rpy="0 0 0" />
+    </collision>
+    <collision>
+      <geometry>
+        <sphere radius="0.064" />
+      </geometry>
+      <origin xyz="0 0 0.049" rpy="0 0 0" />
     </collision>
 <!--inertial-->
@@ -91,14 +87,21 @@
       <material name="${color}" />
     </visual>
-    <!--collision>
-      <geometry>
-        <mesh filename="package://tmr_description/meshes/tm5-900/collision/tm5-900_arm1_c.stl" />
-      </geometry>
-    </collision-->
-    <collision>
-      <geometry>
-        <cylinder length="0.16" radius="0.064" />
-      </geometry>
-      <origin xyz="0 0 -0.145" rpy="0 0 0" />
+    <collision>
+      <geometry>
+        <cylinder length="0.13" radius="0.064" />
+      </geometry>
+      <origin xyz="0 0 -0.130" rpy="0 0 0" />
+    </collision>
+    <collision>
+      <geometry>
+        <sphere radius="0.064" />
+      </geometry>
+      <origin xyz="0 0 -0.065" rpy="0 0 0" />
+    </collision>
+    <collision>
+      <geometry>
+        <sphere radius="0.064" />
+      </geometry>
+      <origin xyz="0 0 -0.195" rpy="0 0 0" />
     </collision>
     <collision>
@@ -110,7 +113,19 @@
     <collision>
       <geometry>
-        <cylinder length="0.16" radius="0.064" />
-      </geometry>
-      <origin xyz="0.429 0 -0.145" rpy="0 0 0" />
+        <cylinder length="0.13" radius="0.064" />
+      </geometry>
+      <origin xyz="0.429 0 -0.130" rpy="0 0 0" />
+    </collision>
+    <collision>
+      <geometry>
+        <sphere radius="0.064" />
+      </geometry>
+      <origin xyz="0.429 0 -0.065" rpy="0 0 0" />
+    </collision>
+    <collision>
+      <geometry>
+        <sphere radius="0.064" />
+      </geometry>
+      <origin xyz="0.429 0 -0.195" rpy="0 0 0" />
     </collision>
 <!--inertial-->
@@ -134,14 +149,21 @@
       <material name="${color}" />
     </visual>
-    <!--collision>
-      <geometry>
-        <mesh filename="package://tmr_description/meshes/tm5-900/collision/tm5-900_arm2_c.stl" />
-      </geometry>
-    </collision-->
-    <collision>
-      <geometry>
-        <cylinder length="0.095" radius="0.064" />
-      </geometry>
-      <origin xyz="0 0 -0.0193" rpy="0 0 0" />
+    <collision>
+      <geometry>
+        <cylinder length="0.047" radius="0.064" />
+      </geometry>
+      <origin xyz="0 0 -0.0433" rpy="0 0 0" />
+    </collision>
+    <collision>
+      <geometry>
+        <sphere radius="0.064" />
+      </geometry>
+      <origin xyz="0 0 -0.0668" rpy="0 0 0" />
+    </collision>
+    <collision>
+      <geometry>
+        <sphere radius="0.064" />
+      </geometry>
+      <origin xyz="0 0 -0.0198" rpy="0 0 0" />
     </collision>
     <collision>
@@ -153,7 +175,19 @@
     <collision>
       <geometry>
-        <cylinder length="0.118" radius="0.0465" />
-      </geometry>
-      <origin xyz="0.4115 0 -0.0153" rpy="0 0 0" />
+        <cylinder length="0.098" radius="0.0465" />
+      </geometry>
+      <origin xyz="0.4115 0 -0.0253" rpy="0 0 0" />
+    </collision>
+    <collision>
+      <geometry>
+        <sphere radius="0.0465" />
+      </geometry>
+      <origin xyz="0.4115 0 -0.0743" rpy="0 0 0" />
+    </collision>
+    <collision>
+      <geometry>
+        <sphere radius="0.0465" />
+      </geometry>
+      <origin xyz="0.4115 0 0.0237" rpy="0 0 0" />
     </collision>
 <!--inertial-->
@@ -179,18 +213,25 @@
     <!--collision>
       <geometry>
-        <mesh filename="package://tmr_description/meshes/tm5-900/collision/tmr_100w_01_c.stl" />
-      </geometry>
+        <cylinder length="0.049" radius="0.0465" />
+      </geometry>
+      <origin xyz="0 0 0.0245" rpy="0 0 0" />
     </collision-->
     <collision>
       <geometry>
-        <cylinder length="0.049" radius="0.0465" />
-      </geometry>
-      <origin xyz="0 0 0.0245" rpy="0 0 0" />
-    </collision>
-    <collision>
-      <geometry>
-        <cylinder length="0.118" radius="0.0465" />
-      </geometry>
-      <origin xyz="0 0.001 0" rpy="${0.5*pi} 0 0" />
+        <cylinder length="0.096" radius="0.0465" />
+      </geometry>
+      <origin xyz="0 -0.010 0" rpy="${0.5*pi} 0 0" />
+    </collision>
+    <collision>
+      <geometry>
+        <sphere radius="0.0465" />
+      </geometry>
+      <origin xyz="0 0.038 0" rpy="0 0 0" />
+    </collision>
+    <collision>
+      <geometry>
+        <sphere radius="0.0465" />
+      </geometry>
+      <origin xyz="0 -0.058 0" rpy="0 0 0" />
     </collision>
 <!--inertial-->
@@ -216,18 +257,25 @@
     <!--collision>
       <geometry>
-        <mesh filename="package://tmr_description/meshes/tm5-900/collision/tmr_100w_02_c.stl" />
-      </geometry>
+        <cylinder length="0.049" radius="0.0465" />
+      </geometry>
+      <origin xyz="0 0 -0.0245" rpy="0 0 0" />
     </collision-->
     <collision>
       <geometry>
-        <cylinder length="0.049" radius="0.0465" />
-      </geometry>
-      <origin xyz="0 0 -0.0245" rpy="0 0 0" />
-    </collision>
-    <collision>
-      <geometry>
-        <cylinder length="0.118" radius="0.0465" />
-      </geometry>
-      <origin xyz="0 0.001 0" rpy="${0.5*pi} 0 0" />
+        <cylinder length="0.096" radius="0.0465" />
+      </geometry>
+      <origin xyz="0 -0.010 0" rpy="${0.5*pi} 0 0" />
+    </collision>
+    <collision>
+      <geometry>
+        <sphere radius="0.0465" />
+      </geometry>
+      <origin xyz="0 0.038 0" rpy="0 0 0" />
+    </collision>
+    <collision>
+      <geometry>
+        <sphere radius="0.0465" />
+      </geometry>
+      <origin xyz="0 -0.058 0" rpy="0 0 0" />
     </collision>
 <!--inertial-->
@@ -251,14 +299,20 @@
       <material name="${color}" />
     </visual>
-    <!--collision>
-      <geometry>
-        <mesh filename="package://tmr_description/meshes/tm5-900/collision/tmr_ee_c.stl" />
-      </geometry>
-    </collision-->
-    <collision>
-      <geometry>
-        <cylinder length="0.0565" radius="0.0465" />
-      </geometry>
-      <origin xyz="0 0 -0.02825" rpy="0 0 0" />
+    <collision>
+      <geometry>
+        <cylinder length="0.03" radius="0.0465" />
+      </geometry>
+      <origin xyz="0 0 -0.015" rpy="0 0 0" />
+    </collision>
+    <collision>
+      <geometry>
+        <sphere radius="0.0465" />
+      </geometry>
+      <origin xyz="0 0 -0.03" rpy="0 0 0" />
+    </collision>
+    <collision>
+      <geometry>
+        <sphere radius="0.0465" />
+      </geometry>
     </collision>
     <collision>

File: tmr_description/xacro/macro.tm5-900-mesh.urdf.xacro (robot description, xacro)
@@ -24,12 +24,7 @@
       <material name="${color}" />
     </visual>
-    <!--collision>
+    <collision>
       <geometry>
         <mesh filename="package://tmr_description/meshes/tm5-900/collision/tm5_base_c.stl" />
-      </geometry>
-    </collision-->
-    <collision>
-      <geometry>
-        <sphere radius="0.09" />
       </geometry>
     </collision>
@@ -54,20 +49,8 @@
       <material name="${color}" />
     </visual>
-    <!--collision>
+    <collision>
       <geometry>
         <mesh filename="package://tmr_description/meshes/tm5-900/collision/tmr_400w_01_c.stl" />
       </geometry>
-    </collision-->
-    <collision>
-      <geometry>
-        <cylinder length="0.16" radius="0.064" />
-      </geometry>
-      <origin xyz="0 0 -0.001" rpy="0 0 0" />
-    </collision>
-    <collision>
-      <geometry>
-        <cylinder length="0.066" radius="0.064" />
-      </geometry>
-      <origin xyz="0 -0.033 0" rpy="${-0.5*pi} 0 0" />
     </collision>
 <!--inertial-->
@@ -91,26 +74,8 @@
       <material name="${color}" />
     </visual>
-    <!--collision>
+    <collision>
       <geometry>
         <mesh filename="package://tmr_description/meshes/tm5-900/collision/tm5-900_arm1_c.stl" />
       </geometry>
-    </collision-->
-    <collision>
-      <geometry>
-        <cylinder length="0.16" radius="0.064" />
-      </geometry>
-      <origin xyz="0 0 -0.145" rpy="0 0 0" />
-    </collision>
-    <collision>
-      <geometry>
-        <cylinder length="0.429" radius="0.06" />
-      </geometry>
-      <origin xyz="0.2145 0 -0.146" rpy="0 ${0.5*pi} 0" />
-    </collision>
-    <collision>
-      <geometry>
-        <cylinder length="0.16" radius="0.064" />
-      </geometry>
-      <origin xyz="0.429 0 -0.145" rpy="0 0 0" />
     </collision>
 <!--inertial-->
@@ -122,5 +87,5 @@
     <parent link="${prefix}link_2" />
     <child link="${prefix}link_3" />
-    <origin xyz="0.429 0 0" rpy="0 0 0" />
+    <origin  xyz="0.429 0 0" rpy="0 0 0" />
     <axis xyz="0 0 1" />
 <!--limit-->
@@ -134,26 +99,8 @@
       <material name="${color}" />
     </visual>
-    <!--collision>
+    <collision>
       <geometry>
         <mesh filename="package://tmr_description/meshes/tm5-900/collision/tm5-900_arm2_c.stl" />
       </geometry>
-    </collision-->
-    <collision>
-      <geometry>
-        <cylinder length="0.095" radius="0.064" />
-      </geometry>
-      <origin xyz="0 0 -0.0193" rpy="0 0 0" />
-    </collision>
-    <collision>
-      <geometry>
-        <cylinder length="0.4115" radius="0.044" />
-      </geometry>
-      <origin xyz="0.20575 0 -0.0163" rpy="0 ${0.5*pi} 0" />
-    </collision>
-    <collision>
-      <geometry>
-        <cylinder length="0.118" radius="0.0465" />
-      </geometry>
-      <origin xyz="0.4115 0 -0.0153" rpy="0 0 0" />
     </collision>
 <!--inertial-->
@@ -177,20 +124,8 @@
       <material name="${color}" />
     </visual>
-    <!--collision>
+    <collision>
       <geometry>
         <mesh filename="package://tmr_description/meshes/tm5-900/collision/tmr_100w_01_c.stl" />
       </geometry>
-    </collision-->
-    <collision>
-      <geometry>
-        <cylinder length="0.049" radius="0.0465" />
-      </geometry>
-      <origin xyz="0 0 0.0245" rpy="0 0 0" />
-    </collision>
-    <collision>
-      <geometry>
-        <cylinder length="0.118" radius="0.0465" />
-      </geometry>
-      <origin xyz="0 0.001 0" rpy="${0.5*pi} 0 0" />
     </collision>
 <!--inertial-->
@@ -214,20 +149,8 @@
       <material name="${color}" />
     </visual>
-    <!--collision>
+    <collision>
       <geometry>
         <mesh filename="package://tmr_description/meshes/tm5-900/collision/tmr_100w_02_c.stl" />
       </geometry>
-    </collision-->
-    <collision>
-      <geometry>
-        <cylinder length="0.049" radius="0.0465" />
-      </geometry>
-      <origin xyz="0 0 -0.0245" rpy="0 0 0" />
-    </collision>
-    <collision>
-      <geometry>
-        <cylinder length="0.118" radius="0.0465" />
-      </geometry>
-      <origin xyz="0 0.001 0" rpy="${0.5*pi} 0 0" />
     </collision>
 <!--inertial-->
@@ -251,20 +174,8 @@
       <material name="${color}" />
     </visual>
-    <!--collision>
+    <collision>
       <geometry>
         <mesh filename="package://tmr_description/meshes/tm5-900/collision/tmr_ee_c.stl" />
       </geometry>
-    </collision-->
-    <collision>
-      <geometry>
-        <cylinder length="0.0565" radius="0.0465" />
-      </geometry>
-      <origin xyz="0 0 -0.02825" rpy="0 0 0" />
-    </collision>
-    <collision>
-      <geometry>
-        <box size="0.075 0.064 0.12" />
-      </geometry>
-      <origin xyz="0 0.073 -0.005" rpy="0 0 0" />
     </collision>
 <!--inertial-->
